File: atmega88-breakout.sch (KiCad schematic (older format))
At the start: 10 parts, among them J1 Conn_01x08_Male, J2 ICSP Header, J4 Conn_01x08_Male, U1 ATmega88PA-AU

Commit message: Route all IO, add user LED, need to add power headers
Parts:
- added D1: LED_Small, LED_SMD:LED_0805_2012Metric, symbol Device:LED_Small
- added R1: R_Small, Resistor_SMD:R_0805_2012Metric, symbol Device:R_Small
- U1: symbol MCU_Microchip_ATmega:ATmega88PA-AU -> atmega88-breakout-rescue:ATmega88PA-AU-MCU_Microchip_ATmega
Connections:
- net D0: now also R1.1
- net GND: now also D1.1 (K)
- new net: D1.2 (A), R1.2
Changed lines of the file:
@@
 EESchema Schematic File Version 4
-EELAYER 30 0
+LIBS:atmega88-breakout-cache
+EELAYER 26 0
 EELAYER END
 $Descr A4 11693 8268
@@
 Comment4 ""
 $EndDescr
-Entry Wire Line
-	-1150 550  -1050 650
-$Comp
-L MCU_Microchip_ATmega:ATmega88PA-AU U1
+$Comp
+L atmega88-breakout-rescue:ATmega88PA-AU-MCU_Microchip_ATmega U1
 U 1 1 5FC75EB9
 P 5200 4000
@@
 Text Label 5900 5200 0    50   ~ 0
 D7
-Wire Wire Line
-	5800 4500 6050 4500
 Wire Wire Line
 	6050 4600 5800 4600
@@
 NoConn ~ 7500 3250
 NoConn ~ 7500 3350
+$Comp
+L Device:R_Small R1
+U 1 1 5FE27389
+P 6350 4850
+F 0 "R1" H 6409 4896 50  0000 L CNN
+F 1 "R_Small" H 6409 4805 50  0000 L CNN
+F 2 "Resistor_SMD:R_0805_2012Metric" H 6350 4850 50  0001 C CNN
+F 3 "~" H 6350 4850 50  0001 C CNN
+	1    6350 4850
+	1    0    0    -1
+$EndComp
+$Comp
+L Device:LED_Small D1
+U 1 1 5FE274C0
+P 6350 5100
+F 0 "D1" V 6396 5032 50  0000 R CNN
+F 1 "LED_Small" V 6305 5032 50  0000 R CNN
+F 2 "LED_SMD:LED_0805_2012Metric" V 6350 5100 50  0001 C CNN
+F 3 "~" V 6350 5100 50  0001 C CNN
+	1    6350 5100
+	0    -1   -1   0
+$EndComp
+$Comp
+L power:GND #PWR08
+U 1 1 5FE2758A
+P 6350 5250
+F 0 "#PWR08" H 6350 5000 50  0001 C CNN
+F 1 "GND" H 6355 5077 50  0000 C CNN
+F 2 "" H 6350 5250 50  0001 C CNN
+F 3 "" H 6350 5250 50  0001 C CNN
+	1    6350 5250
+	1    0    0    -1
+$EndComp
+Wire Wire Line
+	6350 5250 6350 5200
+Wire Wire Line
+	6350 5000 6350 4950
+Wire Wire Line
+	6350 4500 6350 4750
+Wire Wire Line
+	5800 4500 6350 4500
 Wire Bus Line
 	6450 3800 6450 4550

Commit message: Rev A release (ordered)
Parts:
- removed J1, J4: Conn_01x08_Male, Connector_PinHeader_2.54mm:PinHeader_1x08_P2.54mm_Vertical, symbol Connector:Conn_01x08_Male
- added J1, J3: Conn_01x09, Connector_PinHeader_2.54mm:PinHeader_1x09_P2.54mm_Vertical, symbol Connector_Generic:Conn_01x09
- added TP1, TP2, TP3, TP4, TP5, TP6, TP7, TP8: TestPoint, TestPoint:TestPoint_Pad_D1.5mm, symbol Connector:TestPoint
- C1: footprint Capacitor_Tantalum_SMD:CP_EIA-3528-12_Kemet-T -> Capacitor_Tantalum_SMD:CP_EIA-3216-18_Kemet-A
- R1: value R_Small -> 1k
Connections:
- net AREF is gone; now on net VAA: U1.20 (AREF)
- net ADC6: now also J1.1 (Pin_1)
- net B0: now also TP1.1
- net B1: now also TP2.1
- net B2: now also TP3.1
- net B3: now also TP4.1
- net B4: now also TP5.1
- net B5: now also TP6.1
- net B6: now also TP7.1
- net B7: now also TP8.1
- net C0: now also J1.2 (Pin_2)
- net C1: now also J1.3 (Pin_3)
- net C2: now also J1.4 (Pin_4)
- net C3: now also J1.5 (Pin_5)
- net C4: now also J1.6 (Pin_6)
- net C5: now also J1.7 (Pin_7)
- net C6: now also J1.8 (Pin_8)
- net D0: now also J3.8 (Pin_8)
- net D1: now also J3.7 (Pin_7)
- net D2: now also J3.6 (Pin_6)
- net D3: now also J3.5 (Pin_5)
- net D4: now also J3.4 (Pin_4)
- net D5: now also J3.3 (Pin_3)
- net D6: now also J3.2 (Pin_2)
- net D7: now also J3.1 (Pin_1)
- net GND: now also J1.9 (Pin_9)
- net VCC: now also J3.9 (Pin_9)
- no-connect marks 8 -> 0
Other:
- moved on the sheet: C1, C2, C3, C4, D1, J2, JP1, L1, R1, U1
